File: pcb/7001-mainboard/7001-ventilator_mainboard.sch (KiCad schematic (older format))
At the start: 87 parts, among them J1 USB_B_Micro, J10 UART, J2 SWD, J3 Conn_01x02_MountingPin, J4 DNI, J5 24VIN, J6 5V out, J7 PREG_PWR, J8 PREG_SIGNALS, J9 Raspberry_Pi_2_3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

Commit message: schematics: ready for review?
Parts:
- removed C18: 1uF, Capacitor_SMD:C_0805_2012Metric, symbol Device:C
- removed C19: 2.2nF, Capacitor_SMD:C_0805_2012Metric, symbol Device:C
- removed D1: BZT52C10+, Diode_SMD:D_SOD-123, symbol Diode:BZT52Bxx
- removed J3: Conn_01x02_MountingPin, Jitter_Footprints:JST_ZH_S2B-ZR-SM4A-TF_1x02-1MP_P1.5mm_Horizontal, symbol Connector_Generic_MountingPin:Conn_01x02_MountingPin
- removed Q1: IRLML6244TRPbF, Package_TO_SOT_SMD:SOT-23, symbol Device:Q_NMOS_GSD
- removed R6: 1k, Resistor_SMD:R_0805_2012Metric, symbol Device:R
- removed R7: 4.7k, Resistor_SMD:R_0805_2012Metric, symbol Device:R
- removed TP10: valve_2_fet, TestPoint:TestPoint_Pad_D1.0mm, symbol Connector:TestPoint
- added C42, C44: 10uF 50V, Capacitor_SMD:C_1206_3216Metric, symbol Device:C
- added C45: 2.2nF 50V, Capacitor_SMD:C_0805_2012Metric, symbol Device:C
- added D1, D2: D_Schottky, Diode_SMD:D_SOD-123F, symbol Device:D_Schottky
- added J13, J14: PREG_PWR, Jitter_Footprints:TerminalBlock_Wurth_WR-TBL_691322110002_1x02_P3.50mm_Horizontal, symbol Connector_Generic:Conn_01x02
- added R33, R35: 1k5, Resistor_SMD:R_0805_2012Metric, symbol Device:R
- added R34, R36: 4.7k, Resistor_SMD:R_0805_2012Metric, symbol Device:R
- added U13, U14: ITS4142NHUMA1, Package_TO_SOT_SMD:SOT-223, symbol Jitter_Components:ITS4142NHUMA1
- C17: value 2.2nF -> 2.2nF 50V
- gave numbers to parts that had none: 20
Connections:
- net labels added: 24V_SW1_OUT, 24V_SW2_OUT, switch_1_out, switch_2_out
- net labels removed: +6V
- wire segments 238 -> 254
Other:
- note added: "4-20mA DAC to controll\nthe pressure regulator.\nThe regulator also gives\na feedback signal 4-20mA.\n\nThe feedback is not used\ndirectly for control, but\ncan be used as sanity check."
- note added: "5V power is provided\nfor the Raspberry Pi\nvia this connector.\nUART is also connected.\n\nAs a fallback, the Pi\ncan use its own PSU and\nconnect via USB."
- note added: "ESD protection\nSee datasheet for layout\n\nNote: USB is optional:\n- debugging (UART-over-USB)\n- raspberry pi (alt voor connector)\n"
- note added: "NOTE: LPC11u is 3.3V but 5v-tolerant for I2C,\noptional I2C-based flow sensors allow 2.5V as digital high\npressure sensor is 3.3V-based, unknown if 5V-tolerant"
- note added: "RPI connector"
- note added: "TODO\n\n- test points\n- ADC in header\n- GPIO header"
- note removed: "Actuator control"
- note removed: "CT16B0_MAT0"
- note removed: "ESD protection\n\nSee datasheet for layout"
- note removed: "Mogelijk handige copy-paste bouwblokjes"
- note removed: "NOTE: LPC11u is 5v-tolerant for I2C,\nflow sensors are 5V-based, but allow 2.5V as digital high,\npressure sensor is 3.3V-based, unknown if 5V-tolerant"
- note removed: "Pull-down resistors: Actuators should be off by default.\n\nWhen the firmware is not running (for example during an update),\nthe microcontroller pins have a 85uA pull-up current enabled.\nThis would cause the actuators to start running unintentionally,\nWe avoid this by placing a strong pull-down resistor:\nR_pulldown = (0.5V/85uA) -> R_puldown < 5.6k"
- note removed: "RPI hat"
- note removed: "TODO\nWith prototype: tune gate resistor value\nHigher = lower EMC, too high = slow response"
- note removed: "TODO\n\n- extra on/off outputs (voltage? maybe relays?)\n- test points\n- ADC in header\n- GPIO header"
- note removed: "pwm out?"
- moved on the sheet: C1, C17, J1, U2
