File: pcb/7001-mainboard/7001-ventilator_mainboard.sch (KiCad schematic (older format))
At the start: 117 parts, among them J1 USB_B_Micro, J10 6-pin header, J11 4-pin screw terminal, J12 3-pin screw terminal, J13 2-pin screw terminal, J14 2-pin screw terminal, J15 2x10-pin header, J16 10-pin SWD header, J2 4-pin header, J3 2-pin screw terminal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

Commit message: update layout
Connections:
- net LED_ERROR: now also U3.42 (PIO0_23); no longer U3.10 (PIO0_2)
- net LED_STATUS: now also U3.45 (PIO0_17); no longer U3.9 (PIO0_20)
- net MCU_IO_1: no longer U3.1 (PIO1_25)
- net MCU_IO_2: now also U3.48 (PIO1_16); no longer U3.47 (PIO0_19)
- net MCU_IO_3: now also U3.47 (PIO0_19); no longer U3.46 (PIO0_18)
- net MCU_IO_4: now also U3.46 (PIO0_18); no longer U3.45 (PIO0_17)
- net PREG_CLEAR: now also U3.23 (PIO0_7); no longer U3.42 (PIO0_23)
- net PSENSE_1_DATA_READY: now also U3.40 (PIO0_16); no longer U3.23 (PIO0_7)
- net PSENSE_1_SPI_~CS~: now also U3.2 (PIO1_19); no longer U3.22 (PIO0_6)
- net PSENSE_2_SPI_~CS~: now also U3.1 (PIO1_25); no longer U3.21 (PIO1_24)
- net ~ISP~: now also J4.3 (Pin_3); no longer J4.2 (Pin_2)
- net ~RESET~: now also J4.2 (Pin_2); no longer J4.3 (Pin_3)
Other:
- moved on the sheet: J4
Changed lines of the file:
@@
 	5500 7850 6000 7850
 Wire Wire Line
-	4100 6750 2850 6750
+	4100 6750 3250 6750
 Wire Wire Line
 	5000 5650 5450 5650
@@
 L Connector_Generic:Conn_01x03 J?
 U 1 1 5E7CEF83
-P 2650 6750
+P 2600 6750
 AR Path="/5BF2E340/5E7CEF83" Ref="J?"  Part="1"
 AR Path="/5E7CEF83" Ref="J4"  Part="1"
-F 0 "J4" H 2650 6450 50  0000 C CNN
-F 1 "DNI" H 2650 6550 50  0000 C CNN
-F 2 "Connector_PinHeader_2.54mm:PinHeader_1x03_P2.54mm_Vertical" H 2650 6750 50  0001 C CNN
-F 3 "~" H 2650 6750 50  0001 C CNN
-	1    2650 6750
+F 0 "J4" H 2600 6450 50  0000 C CNN
+F 1 "DNI" H 2600 6550 50  0000 C CNN
+F 2 "Connector_PinHeader_2.54mm:PinHeader_1x03_P2.54mm_Vertical" H 2600 6750 50  0001 C CNN
+F 3 "~" H 2600 6750 50  0001 C CNN
+	1    2600 6750
 	-1   0    0    1
 $EndComp
@@
 L power:GND #PWR?
 U 1 1 5E7CFA00
-P 2850 6850
+P 2800 6850
 AR Path="/5BF2E340/5E7CFA00" Ref="#PWR?"  Part="1"
 AR Path="/5E7CFA00" Ref="#PWR0150"  Part="1"
-F 0 "#PWR0150" H 2850 6600 50  0001 C CNN
-F 1 "GND" H 2855 6677 50  0000 C CNN
-F 2 "" H 2850 6850 50  0001 C CNN
-F 3 "" H 2850 6850 50  0001 C CNN
-	1    2850 6850
+F 0 "#PWR0150" H 2800 6600 50  0001 C CNN
+F 1 "GND" H 2805 6677 50  0000 C CNN
+F 2 "" H 2800 6850 50  0001 C CNN
+F 3 "" H 2800 6850 50  0001 C CNN
+	1    2800 6850
 	1    0    0    -1
 $EndComp
@@
 ~RESET~
 Wire Wire Line
-	3550 6650 2850 6650
+	3550 6650 3250 6650
 Connection ~ 3550 6650
 Wire Wire Line
@@
 Wire Wire Line
 	4100 8950 3050 8950
-Text Label 3050 8950 0    50   ~ 0
+Text Label 3050 7350 0    50   ~ 0
 PREG_CLEAR
 Text Label 6550 7950 2    50   ~ 0
@@
 Wire Wire Line
 	14150 5750 14400 5750
-Wire Wire Line
-	4100 7250 3050 7250
-Text Label 3050 7250 0    50   ~ 0
+Text Label 6550 7050 2    50   ~ 0
 PSENSE_1_SPI_~CS~
 Wire Wire Line
@@
 Wire Wire Line
 	4100 7350 3050 7350
-Text Label 3050 7350 0    50   ~ 0
+Text Label 3050 8250 0    50   ~ 0
 PSENSE_1_DATA_READY
 Wire Wire Line
@@
 PSENSE_2_DATA_READY
 Wire Wire Line
-	5500 7550 6550 7550
-Text Label 6550 7550 2    50   ~ 0
+	5500 7650 6550 7650
+Text Label 6550 7650 2    50   ~ 0
 PSENSE_2_SPI_~CS~
 Text Label 3600 8850 0    50   ~ 0
@@
 Wire Notes Line
 	8850 11100 8850 9150
-Text Label 3050 8650 0    50   ~ 0
+Text Label 3050 8350 0    50   ~ 0
 LED_STATUS
-Text Label 3050 6850 0    50   ~ 0
+Text Label 3050 8950 0    50   ~ 0
 LED_ERROR
 $Comp
@@
 RPI_IO_3
 Wire Wire Line
-	5500 7650 6550 7650
-Text Label 6550 7650 2    50   ~ 0
-MCU_IO_1
-Wire Wire Line
 	4100 8350 3050 8350
 Wire Wire Line
@@
 Wire Wire Line
 	4100 8550 3050 8550
-Text Label 3050 8550 0    50   ~ 0
+Text Label 6550 6950 2    50   ~ 0
 MCU_IO_2
-Text Label 3050 8450 0    50   ~ 0
+Text Label 3050 8550 0    50   ~ 0
 MCU_IO_3
-Text Label 3050 8350 0    50   ~ 0
+Text Label 3050 8450 0    50   ~ 0
 MCU_IO_4
 Wire Wire Line
@@
 Wire Wire Line
 	3450 6950 3450 7100
-NoConn ~ 5500 6950
-NoConn ~ 5500 7050
-NoConn ~ 4100 8250
 NoConn ~ 4100 8750
 Text Label 7700 1950 0    50   ~ 0
@@
 	4450 10050 4450 9950
 Connection ~ 4450 9950
+Wire Wire Line
+	6550 6950 5500 6950
+NoConn ~ 3050 8650
+Wire Wire Line
+	3050 8250 4100 8250
+NoConn ~ 3050 6850
+NoConn ~ 5500 7550
+Text Label 3050 6750 2    50   ~ 0
+~RESET~
+Wire Wire Line
+	3050 6750 2800 6750
+Text Label 3050 6650 2    50   ~ 0
+~ISP~
+Wire Wire Line
+	3050 6650 2800 6650
+Wire Wire Line
+	5500 7050 6550 7050
 $EndSCHEMATC
