File: pcb/7001-mainboard/7001-ventilator_mainboard.sch (KiCad schematic (older format))
At the start: 143 parts, among them J1 USB_B_Micro, J10 6-pin header, J11 2-pin screw terminal, J13 2-pin screw terminal, J14 2-pin screw terminal, J15 2x10-pin header, J16 10-pin SWD header, J2 6-pin FFC connector, J3 2-pin screw terminal, J4 2-pin screw terminal, J5 2-pin screw terminal, J6 5V out, J7 6-pin FFC connector, J8 2-pin screw terminal, J9 Raspberry_Pi_2_3, Q1 NX3020NAKV,115, U13 ITS4142NHUMA1, U14 ITS4142NHUMA1, U15 MCP4725, U16 LD1086DT33TR, U2 TPD2E2U06, U3 LPC11U37FBD48-401_, U4 MCP1825S-3302E, U5 S24SE05004PDFA_DC-DC, U6 MCP4725, U7 ITS4142NHUMA1, Y1 12MHz

Commit message: PCB layout: final locations and BOM (?)
Parts:
- J11, J8: value 2-pin screw terminal -> 5-pin screw terminal; Farnell 1841318 -> (none)
- J5: value 2-pin screw terminal -> 5-pin screw terminal vertical; footprint Jitter_Footprints:TerminalBlock_Wurth_WR-TBL_691322110008_1x08_P3.50mm_Horizontal -> Jitter_Footprints:TerminalBlock_Wurth_WR-TBL_691321100005_1x05_P3.50mm_Vertical; symbol Connector_Generic:Conn_01x08 -> Connector_Generic:Conn_01x05; Farnell 1841314 -> (none); MPN 691321100008 -> 691321100005
- U16: value LD1086DT33TR -> LD1086DTTR; Farnell 1467774 -> (none); MPN LD1086DT33TR -> LD1086DTTR (adjustable)
Connections:
- net GND: no longer J5.1 (Pin_1), J5.2 (Pin_2)
- net UPS_DISCHG: now reaches R12.1
- net UPS_DISCHG: now also J5.4 (Pin_4); no longer J5.5 (Pin_5)
- net PWR-: now reaches C46.2, D4.1 (A1), FL1.1, RV1.2
- net PWR-: now also J5.1 (Pin_1); no longer J5.3 (Pin_3)
- net PWR+: now reaches C46.1, D4.2 (A2), FL1.2, RV1.1
- net PWR+: now also J5.2 (Pin_2); no longer J5.4 (Pin_4)
- net UPS_FAIL: now reaches R22.1
- net UPS_FAIL: now also J5.5 (Pin_5); no longer J5.7 (Pin_7)
- net 24_CHOKE: now reaches C47.1, D3.2 (A), FL1.4
- new net UPS_3V3_PU: J5.3 (Pin_3), R23.1
Other:
- note removed: "BATT_DISCHG"
- note removed: "BATT_FAIL"
- note removed: "NOTE: this is \na vertical\nheader!\n3D Footprint\nis wrong.."
- note removed: "PSU_EARTH"
- note removed: "TODO 6-pins?"
- note removed: "TODO Earth:\ndirectly to GND?"
- note removed: "TODO REVIEW FOOTPRINT\nNOTE: LDO may run hot!"
- moved on the sheet: R23
Changed lines of the file:
@@
 Text Notes 3700 5350 0    79   ~ 16
 5V -> 3.3V
-$Comp
-L Connector_Generic:Conn_01x08 J?
-U 1 1 5EBE6F1F
-P 650 2150
-AR Path="/5BF2E340/5EBE6F1F" Ref="J?"  Part="1"
-AR Path="/5EBE6F1F" Ref="J5"  Part="1"
-F 0 "J5" H 650 2600 50  0000 C CNN
-F 1 "2-pin screw terminal" H 650 1950 50  0001 C CNN
-F 2 "Jitter_Footprints:TerminalBlock_Wurth_WR-TBL_691322110008_1x08_P3.50mm_Horizontal" H 650 2150 50  0001 C CNN
-F 3 "~" H 650 2150 50  0001 C CNN
-F 4 "691321100008" H 650 2150 50  0001 C CNN "MPN"
-F 5 "1841314" H 650 2150 50  0001 C CNN "Farnell"
-	1    650  2150
-	-1   0    0    1
-$EndComp
 Text Notes 1100 2400 0    50   ~ 0
 24VDC 4A
@@
 $EndComp
 Wire Wire Line
-	2750 2700 2900 2700
-Wire Wire Line
-	2900 2700 2900 2550
+	2750 2700 2750 2550
 Wire Wire Line
 	2750 2900 2900 2900
@@
 	1250 2950 1250 3000
 Wire Wire Line
-	1000 2550 1250 2550
+	1100 2550 1250 2550
 Connection ~ 1250 2550
 Connection ~ 1250 3000
@@
 P 14500 6650
 F 0 "U16" H 14500 6925 50  0000 C CNN
-F 1 "LD1086DT33TR" H 14500 6926 50  0001 C CNN
+F 1 "LD1086DTTR" H 14500 6926 50  0001 C CNN
 F 2 "Package_TO_SOT_SMD:TO-252-2" H 14500 7150 50  0001 C CNN
 F 3 "https://www.st.com/resource/en/datasheet/ld1086.pdf" H 14500 7150 50  0001 C CNN
-F 4 "LD1086DT33TR" H 14500 6650 50  0001 C CNN "MPN"
-F 5 "1467774" H 14500 6650 50  0001 C CNN "Farnell"
+F 4 "LD1086DTTR (adjustable)" H 14500 6650 50  0001 C CNN "MPN"
+F 5 "" H 14500 6650 50  0001 C CNN "Farnell"
 	1    14500 6650
 	1    0    0    -1
@@
 	1    0    0    1
 $EndComp
-Text Notes 16150 6350 0    59   ~ 12
-TODO REVIEW FOOTPRINT\nNOTE: LDO may run hot!
 Text Notes 16150 8700 0    59   ~ 12
 TODO VERIFY\nFFC pinout\nmatches flow sensor
@@
 	3050 3000 3150 3000
 Wire Wire Line
-	3050 2550 2900 2550
+	3050 2550 2750 2550
 Connection ~ 3050 2550
 Wire Wire Line
@@
 AR Path="/60E8C3C0" Ref="J11"  Part="1"
 F 0 "J11" H 15800 4150 50  0000 C CNN
-F 1 "2-pin screw terminal" H 15800 4250 50  0001 C CNN
+F 1 "5-pin screw terminal" H 15800 4250 50  0001 C CNN
 F 2 "Jitter_Footprints:TerminalBlock_Wurth_WR-TBL_691322110005_1x05_P3.50mm_Horizontal" H 15800 4450 50  0001 C CNN
 F 3 "~" H 15800 4450 50  0001 C CNN
 F 4 "691322110005" H 15800 4450 50  0001 C CNN "MPN"
-F 5 "1841318" H 15800 4450 50  0001 C CNN "Farnell"
 	1    15800 4450
 	1    0    0    1
@@
 AR Path="/61520C02" Ref="J8"  Part="1"
 F 0 "J8" H 15800 1800 50  0000 C CNN
-F 1 "2-pin screw terminal" H 15800 1900 50  0001 C CNN
+F 1 "5-pin screw terminal" H 15800 1900 50  0001 C CNN
 F 2 "Jitter_Footprints:TerminalBlock_Wurth_WR-TBL_691322110005_1x05_P3.50mm_Horizontal" H 15800 2100 50  0001 C CNN
 F 3 "~" H 15800 2100 50  0001 C CNN
 F 4 "691322110005" H 15800 2100 50  0001 C CNN "MPN"
-F 5 "1841318" H 15800 2100 50  0001 C CNN "Farnell"
 	1    15800 2100
 	1    0    0    1
@@
 POWER_STATUS_FAIL
 $Comp
-L Device:R R?
-U 1 1 6173E463
-P 1300 1600
-AR Path="/5BF2E340/6173E463" Ref="R?"  Part="1"
-AR Path="/6173E463" Ref="R23"  Part="1"
-F 0 "R23" H 1150 1450 50  0000 L CNN
-F 1 "1k5" H 1100 1550 50  0000 L CNN
-F 2 "Resistor_SMD:R_0805_2012Metric" V 1230 1600 50  0001 C CNN
-F 3 "~" H 1300 1600 50  0001 C CNN
-	1    1300 1600
-	-1   0    0    1
-$EndComp
-$Comp
-L power:+3.3V #PWR0215
-U 1 1 6173E469
-P 1300 1450
-F 0 "#PWR0215" H 1300 1300 50  0001 C CNN
-F 1 "+3.3V" H 1315 1623 50  0000 C CNN
-F 2 "" H 1300 1450 50  0001 C CNN
-F 3 "" H 1300 1450 50  0001 C CNN
-	1    1300 1450
-	1    0    0    -1
-$EndComp
-$Comp
 L power:GND #PWR0216
 U 1 1 6173E46F
@@
 	0    -1   -1   0
 $EndComp
-Text Notes 850  1850 0    50   ~ 0
-BATT_FAIL
-Text Notes 850  2050 0    50   ~ 0
-BATT_DISCHG
 Text Label 6500 8100 2    50   ~ 0
 POWER_STATUS_DISCHARGING
@@
 	3550 7400 3550 7600
 Wire Wire Line
-	1000 2550 1000 2150
-Wire Wire Line
-	1000 2150 850  2150
-Wire Wire Line
-	1900 1850 1900 2050
+	1100 2550 1100 2150
 Wire Wire Line
-	1900 2050 850  2050
+	1100 2150 800  2150
 Wire Wire Line
-	1900 1850 2600 1850
-Wire Wire Line
-	850  1850 1800 1850
+	800  1850 1800 1850
 Wire Wire Line
 	1800 1850 1800 1000
@@
 	1800 1000 2600 1000
 Wire Wire Line
-	1300 1750 850  1750
-$Comp
-L power:GND #PWR?
-U 1 1 61E31F80
-P 850 2900
-AR Path="/5BF2E340/61E31F80" Ref="#PWR?"  Part="1"
-AR Path="/61E31F80" Ref="#PWR0217"  Part="1"
-F 0 "#PWR0217" H 850 2650 50  0001 C CNN
-F 1 "GND" H 855 2727 50  0000 C CNN
-F 2 "" H 850 2900 50  0001 C CNN
-F 3 "" H 850 2900 50  0001 C CNN
-	1    850  2900
-	-1   0    0    -1
-$EndComp
-Wire Wire Line
-	850  2250 950  2250
+	800  2250 1000 2250
 Wire Wire Line
-	950  2250 950  3000
+	1000 2250 1000 3000
 Wire Wire Line
-	950  3000 1250 3000
-Wire Wire Line
-	850  2350 850  2450
-Connection ~ 850  2450
-Wire Wire Line
-	850  2450 850  2900
-Text Notes 350  2700 2    50   ~ 0
-TODO Earth:\ndirectly to GND?
-Text Notes 850  2900 1    50   ~ 0
-PSU_EARTH
-Text Notes 350  2150 2    50   ~ 0
-NOTE: this is \na vertical\nheader!\n3D Footprint\nis wrong..
-Text Notes 350  2450 2    50   ~ 0
-TODO 6-pins?
+	1000 3000 1250 3000
 $Comp
 L power:GND #PWR?
@@
 Wire Wire Line
 	15700 8050 15700 8150
-Wire Wire Line
-	850  1950 1300 1950
-Wire Wire Line
-	1300 1950 1300 1750
-Connection ~ 1300 1750
 Text Label 3000 9700 0    50   ~ 0
 LED_ERROR
@@
 Wire Wire Line
 	12200 9150 12350 9150
+$Comp
+L Connector_Generic:Conn_01x05 J?
+U 1 1 5EBE6F1F
+P 600 2050
+AR Path="/5BF2E340/5EBE6F1F" Ref="J?"  Part="1"
+AR Path="/5EBE6F1F" Ref="J5"  Part="1"
+F 0 "J5" H 600 2400 50  0000 C CNN
+F 1 "5-pin screw terminal vertical" H 600 1850 50  0001 C CNN
+F 2 "Jitter_Footprints:TerminalBlock_Wurth_WR-TBL_691321100005_1x05_P3.50mm_Vertical" H 600 2050 50  0001 C CNN
+F 3 "~" H 600 2050 50  0001 C CNN
+F 4 "691321100005" H 600 2050 50  0001 C CNN "MPN"
+	1    600  2050
+	-1   0    0    1
+$EndComp
+$Comp
+L power:+3.3V #PWR0215
+U 1 1 6173E469
+P 1350 1450
+F 0 "#PWR0215" H 1350 1300 50  0001 C CNN
+F 1 "+3.3V" H 1365 1623 50  0000 C CNN
+F 2 "" H 1350 1450 50  0001 C CNN
+F 3 "" H 1350 1450 50  0001 C CNN
+	1    1350 1450
+	1    0    0    -1
+$EndComp
+$Comp
+L Device:R R?
+U 1 1 6173E463
+P 1350 1600
+AR Path="/5BF2E340/6173E463" Ref="R?"  Part="1"
+AR Path="/6173E463" Ref="R23"  Part="1"
+F 0 "R23" H 1200 1450 50  0000 L CNN
+F 1 "1k5" H 1150 1550 50  0000 L CNN
+F 2 "Resistor_SMD:R_0805_2012Metric" V 1280 1600 50  0001 C CNN
+F 3 "~" H 1350 1600 50  0001 C CNN
+	1    1350 1600
+	-1   0    0    1
+$EndComp
+Wire Wire Line
+	1350 2050 1350 1750
+Wire Wire Line
+	2100 1950 2100 1850
+Wire Wire Line
+	2100 1850 2600 1850
+Text Label 800  2150 0    50   ~ 0
+PWR+
+Text Label 800  2250 0    50   ~ 0
+PWR-
+Wire Wire Line
+	800  1950 2100 1950
+Text Label 800  2050 0    50   ~ 0
+UPS_3V3_PU
+Wire Wire Line
+	800  2050 1350 2050
+Text Label 800  1950 0    50   ~ 0
+UPS_DISCHG
+Text Label 800  1850 0    50   ~ 0
+UPS_FAIL
+Text Label 2750 2550 0    50   ~ 0
+24_CHOKE
 $EndSCHEMATC
