File: pcb/7001-mainboard/7001-ventilator_mainboard.kicad_pcb (KiCad board)
At the start: 2 copper layers, 98.5 x 110 mm, 148 parts, among them J1 USB_B_Micro, J10 6-pin header, J11 4-pin screw terminal, J12 3-pin screw terminal, J13 2-pin screw terminal, J14 2-pin screw terminal, J15 2x10-pin header, J16 10-pin SWD header, J2 4-pin header, J3 2-pin screw terminal, J4 DNI, J5 2-pin screw terminal, J6 5V out, J7 2-pin screw terminal, J8 3-pin screw terminal, J9 Raspberry_Pi_2_3, U1 MPRLS0001PG0000SA, U10 ABPMAND001PG2A3, U11 MPVZ5010GW6U, U12 MPVZ5010GW6U, U13 ITS4142NHUMA1, U14 ITS4142NHUMA1, U2 TPD2E2U06, U3 LPC11U37FBD48-401_, U4 MCP1825S-3302E, U5 S24SE05004PDFA_DC-DC, U6 LM2937IMP-12/NOPB, U7 AD5410AREZ, U8 MPRLS0001PG0000SA, U9 ABPMAND001PG2A3, Y1 12MHz

Commit message: layout: everything except pressure sensors
Routing:
- net +5V: track 129.9 -> 151.2 mm, vias 2 -> 4
- net /I2C_SDA: track 99.4 -> 110.8 mm
- net /PSENSE_SPI_MISO: track 29.9 -> 40.6 mm
- net /I2C_SCL: track 100.5 -> 111.0 mm
- net /~RESET~: track 86.3 -> 90.4 mm
- net GND: track 226.8 -> 230.4 mm, vias 132 -> 135
- net /PSENSE_2_SPI_~CS~: track 16.4 -> 18.7 mm
- net /switch_2_out: track 73.4 -> 75.1 mm
- net /PREG_SPI_MOSI: track 81.7 -> 83.3 mm
- net /~ISP~: track 33.6 -> 35.1 mm
- net /PSENSE_SPI_CLK: track 27.2 -> 26.1 mm
- net Net-(D10-Pad2): track 1.33 -> 2.21 mm
- net /PSENSE_SPI_MOSI: track 23.4 -> 24.2 mm

Commit message: Fix footprint bugs
Parts:
- added FID1: DNI, Fiducial:Fiducial_1mm_Mask2mm, F.Cu at (82.0, 207.0)
- added FID2: DNI, Fiducial:Fiducial_1mm_Mask2mm, F.Cu at (150.0, 207.0)
- added FID3: DNI, Fiducial:Fiducial_1mm_Mask2mm, F.Cu at (102.0, 117.0)
- added FID4: DNI, Fiducial:Fiducial_1mm_Mask2mm, F.Cu at (163.0, 117.0)
- added FID5: DNI, Fiducial:Fiducial_1mm_Mask2mm, F.Cu at (70.0, 157.0)
- C22: footprint Jitter_Footprints:CP_Elec_12.5x13.5 -> Jitter_Footprints:CP_Elec_12.5_MAL214699107E3
- J1: footprint Connector_USB:USB_Micro-B_Molex_47346-0001 -> Jitter_Footprints:USB_Micro-B_Molex_47346-0001
- moved U1 41.7 mm to (178.6, 153.6), turned to 270 degrees
- moved J1 1.20 mm to (102.8, 143.4)
- moved D4 0.60 mm to (158.2, 197.5)
- moved RV1 0.60 mm to (158.2, 194.0)
- moved C47 0.45 mm to (158.1, 176.5)
Routing:
- net /PSENSE_RESET: track 49.4 -> 28.8 mm
- net /PSENSE_2_SPI_~CS~: track 18.7 -> 39.3 mm
- net GND: track 230.4 -> 242.0 mm
- net /PSENSE_2_DATA_READY: track 34.8 -> 44.2 mm
- net /PSENSE_SPI_MOSI: track 24.2 -> 14.7 mm
- net +24V: track 173.6 -> 168.3 mm
- net /switch_1_out: track 93.6 -> 96.8 mm

Commit message: PCB: Finish layout
Parts:
- moved TP3 67.9 mm to (142.0, 142.8)
- moved R24 62.8 mm to (147.7, 126.4), turned to 270 degrees
- moved C35 60.0 mm to (143.5, 124.6), turned to 270 degrees
- moved R1 56.1 mm to (148.3, 123.5)
- moved R20 52.5 mm to (145.5, 124.6), turned to 90 degrees
- moved R22 51.1 mm to (162.3, 137.8), turned to 270 degrees
- moved U9 49.6 mm to (154.8, 135.9), turned to 270 degrees
- moved C34 47.3 mm to (151.8, 123.5)
- moved C5 42.5 mm to (151.5, 134.6), turned to 90 degrees
- moved C8 32.5 mm to (162.3, 134.4), turned to 270 degrees
- moved C31 31.0 mm to (155.2, 123.5), turned to 180 degrees
- moved U1 30.1 mm to (155.3, 134.6)
- moved C30 25.9 mm to (155.2, 121.5), turned to 180 degrees
- moved R25 14.2 mm to (145.8, 150.7)
- moved TP2 12.3 mm to (136.9, 134.5)
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Connections:
- U3 pad 1: /PSENSE_2_SPI_~CS~ -> /PSENSE_1_DATA_READY
- U3 pad 34: /A_PRESSURE_1 -> /A_PRESSURE_2
- U3 pad 35: /A_PRESSURE_2 -> /A_PRESSURE_1
- U3 pad 40: /PSENSE_1_DATA_READY -> /PSENSE_2_SPI_~CS~
Routing:
- net +5V: track 151.2 -> 255.1 mm, vias 4 -> 8
- net +3V3: track 204.5 -> 295.0 mm, vias 6 -> 9
- net /PSENSE_SPI_MOSI: track 14.7 -> 87.0 mm, vias 2 -> 4
- net /PSENSE_RESET: track 28.8 -> 88.1 mm, vias 2 -> 4
- net /PSENSE_SPI_MISO: track 40.6 -> 99.7 mm, vias 2 -> 6
- net /PSENSE_SPI_CLK: track 26.1 -> 77.3 mm, vias 2 -> 4
- net /PSENSE_2_DATA_READY: track 44.2 -> 87.6 mm, vias 2 -> 5
- net /PSENSE_1_DATA_READY: track 13.4 -> 53.0 mm, vias 0 -> 6
- net /PSENSE_1_SPI_~CS~: track 17.0 -> 55.5 mm, vias 2 -> 4
- net /pressure_sensor/P_SDA: track 4.09 -> 41.3 mm, vias 0 -> 2
- net /pressure_sensor/P_SCL: track 4.16 -> 39.6 mm
- net GND: track 242.0 -> 271.6 mm, vias 135 -> 166
- net /A_PRESSURE_1: track 14.3 -> 38.1 mm, vias 2 -> 4
- net /PSENSE_2_SPI_~CS~: track 39.3 -> 61.3 mm
- net /A_PRESSURE_2: track 11.6 -> 32.3 mm, vias 2 -> 3
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Other:
- board text removed: "TODO double-check bouard outline+header pinout is mirrored corerctly !"
