File: pcb/7001-mainboard/pressure_sensor.sch (KiCad schematic (older format))
At the start: 31 parts, among them U1 MPRLS0001PG0000SA, U10 ABPMAND001PG2A3, U11 MPVZ5010GW6U, U12 MPVZ5010GW6U, U8 MPRLS0001PG0000SA, U9 ABPMAND001PG2A3

Commit message: PCB: schematics for V2
Parts:
- removed R21: 100k, Resistor_SMD:R_0805_2012Metric, symbol Device:R
- removed R22, R23, R27, R28: 0, Resistor_SMD:R_0805_2012Metric, symbol Device:R
- removed R24, R25, R26: DNI, Resistor_SMD:R_0805_2012Metric, symbol Device:R
- removed U10, U9: ABPMAND001PG2A3, Jitter_Footprints:ABPM+DXXX000XX0XX, symbol Jitter_Components:ABPMXXX000XX0XX
- removed U12: MPVZ5010GW6U, Jitter_Footprints:MPVZ5010GW6U, symbol Sensor_Pressure:MPXH6115A
- added R13: 100k, Resistor_SMD:R_0805_2012Metric, symbol Device:R
- added U9: ABPDXXX000XXAX5, Jitter_Footprints:ABPDXXX000XX0XX, symbol Jitter_Components:ABPDXXX000XXAX5
- C36: value 470pF -> 1nF
Connections:
- net labels added: A_MFC_PRESSURE, A_PSENSE_3, MPVZ5010_OUT
- net labels removed: A_PRESSURE_1, A_PRESSURE_2, I2C_SCL, I2C_SDA, MPVZ5010_1_OUT, MPVZ5010_2_OUT, P_SCL, P_SDA
- wire segments 74 -> 43
- no-connect marks 6 -> 7
Other:
- note added: "5V to 3V divider +\nRC filter: Fc = 1.8Khz\n"
- note added: "Pressure after patient (0-70mbar)"
- note added: "Pressure before patient (0-70mbar)"
- note added: "Pressure close to patient (0-70mbar)"
- note added: "Pressure sensor 1 (before patient)"
- note added: "Pressure sensor 2 (after patient)"
- note added: "Pressure sensor 3 (weaning)"
- note added: "Pressure sensor 4 (MFC output)"
- note added: "Pressure vessel between MFC\nand pressure regulator (0.5-1 bar)"
- note removed: "5V to 3V divider.\nRC filter: 40kOhm, 2.2nF: Fc= 1.8Khz\n"
- note removed: "ABP I2c version: U9, R24=DNI, R22,R27,R28=0\nABP analog version: R22,R26,R24=0, R27-28=DNI"
- note removed: "I2C bus\nshared"
- note removed: "NOTE: if placing (multiple)\nI2C sensors, check for\nduplicate addresses!"
- note removed: "Note: place one of the three footprints"
- note removed: "Note: this is optional. Choose at most one of the three footprints"
- note removed: "Pressure sensor 1"
- note removed: "Pressure sensor 2 (optional)"
- moved on the sheet: C30, C31, C34, C35, C5, C6, C8, C9, R1, R20, TP2, U1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
